File: pcb/rabid40/rabid40.kicad_pcb (KiCad board)
At the start: 2 copper layers, 0 parts

Commit message: all components added for the 40
Parts:
- added '1: MX-NoLED, MX_Alps_Hybrid:MX-1U-NoLED, F.Cu at (173.8, 138.1)
- added /1: MX-NoLED, MX_Alps_Hybrid:MX-1U-NoLED, F.Cu at (113.2, 138.1)
- added ;1: MX-NoLED, MX_Alps_Hybrid:MX-1U-NoLED, F.Cu at (173.8, 117.9)
- added <1: MX-NoLED, MX_Alps_Hybrid:MX-1U-NoLED, F.Cu at (52.6, 97.7)
- added >1: MX-NoLED, MX_Alps_Hybrid:MX-1U-NoLED, F.Cu at (153.6, 57.3)
- added A1: MX-NoLED, MX_Alps_Hybrid:MX-1U-NoLED, F.Cu at (153.6, 158.3)
- added Alt1: MX-NoLED, MX_Alps_Hybrid:MX-1U-NoLED, F.Cu at (52.6, 138.1)
- added Alt2: MX-NoLED, MX_Alps_Hybrid:MX-1U-NoLED, F.Cu at (133.4, 97.7)
- added B1: MX-NoLED, MX_Alps_Hybrid:MX-1U-NoLED, F.Cu at (93.0, 158.3)
- added C1: 0.1uF, Capacitor_SMD:C_0805_2012Metric, F.Cu at (140.6, 169.9)
- added C2: 0.1uF, Capacitor_SMD:C_0805_2012Metric, F.Cu at (140.6, 172.9)
- added C3: 22pF, Capacitor_SMD:C_0805_2012Metric, F.Cu at (237.2, 75.6)
- added C4: 22pF, Capacitor_SMD:C_0805_2012Metric, F.Cu at (252.5, 58.8)
- added C5: 0.1uF, Capacitor_SMD:C_0805_2012Metric, F.Cu at (258.3, 55.4)
- added C6: 1uF, Capacitor_SMD:C_0805_2012Metric, F.Cu at (49.2, 176.3)
- added C7: 0.1uF, Capacitor_SMD:C_0805_2012Metric, F.Cu at (44.8, 176.3)
- added C8: MX-NoLED, MX_Alps_Hybrid:MX-1U-NoLED, F.Cu at (72.8, 158.3)
- added Caps1: MX-NoLED, MX_Alps_Hybrid:MX-1U-NoLED, F.Cu at (194.0, 117.9)
- added D1: 1N4148W, Diode_SMD:D_SOD-123, F.Cu at (258.9, 48.9)
- added D10: 1N4148W, Diode_SMD:D_SOD-123, F.Cu at (112.5, 173.4)
- added D11: 1N4148W, Diode_SMD:D_SOD-123, F.Cu at (135.5, 173.4)
- added D12: 1N4148W, Diode_SMD:D_SOD-123, F.Cu at (83.7, 173.4)
- added D13: 1N4148W, Diode_SMD:D_SOD-123, F.Cu at (124.0, 173.4)
- added D14: 1N4148W, Diode_SMD:D_SOD-123, F.Cu at (207.0, 107.1)
- added D15: 1N4148W, Diode_SMD:D_SOD-123, F.Cu at (247.4, 52.2)
- added D16: 1N4148W, Diode_SMD:D_SOD-123, F.Cu at (237.9, 72.4)
- added D17: MX-NoLED, MX_Alps_Hybrid:MX-1U-NoLED, F.Cu at (93.0, 138.1)
- added D18: 1N4148W, Diode_SMD:D_SOD-123, F.Cu at (237.9, 69.1)
- added D19: 1N4148W, Diode_SMD:D_SOD-123, F.Cu at (166.6, 149.9)
- added D2: 1N4148W, Diode_SMD:D_SOD-123, F.Cu at (264.7, 48.9)
- added D20: 1N4148W, Diode_SMD:D_SOD-123, F.Cu at (95.2, 170.1)
- added D21: 1N4148W, Diode_SMD:D_SOD-123, F.Cu at (95.2, 173.4)
- added D22: 1N4148W, Diode_SMD:D_SOD-123, F.Cu at (60.7, 173.4)
- added D23: 1N4148W, Diode_SMD:D_SOD-123, F.Cu at (55.0, 173.4)
- added D24: 1N4148W, Diode_SMD:D_SOD-123, F.Cu at (72.2, 170.1)
- added D25: 1N4148W, Diode_SMD:D_SOD-123, F.Cu at (247.4, 55.6)
- added D26: 1N4148W, Diode_SMD:D_SOD-123, F.Cu at (227.2, 82.7)
- added D27: 1N4148W, Diode_SMD:D_SOD-123, F.Cu at (78.0, 173.4)
- added D28: 1N4148W, Diode_SMD:D_SOD-123, F.Cu at (129.7, 173.4)
- added D29: 1N4148W, Diode_SMD:D_SOD-123, F.Cu at (89.5, 170.1)
- added D3: 1N4148W, Diode_SMD:D_SOD-123, F.Cu at (253.2, 52.2)
- added D30: 1N4148W, Diode_SMD:D_SOD-123, F.Cu at (60.7, 170.1)
- added D31: 1N4148W, Diode_SMD:D_SOD-123, F.Cu at (101.0, 170.1)
- added D32: 1N4148W, Diode_SMD:D_SOD-123, F.Cu at (253.2, 55.6)
- added D33: 1N4148W, Diode_SMD:D_SOD-123, F.Cu at (135.5, 170.1)
- added D34: 1N4148W, Diode_SMD:D_SOD-123, F.Cu at (101.0, 173.4)
- added D35: 1N4148W, Diode_SMD:D_SOD-123, F.Cu at (118.2, 173.4)
- added D36: 1N4148W, Diode_SMD:D_SOD-123, F.Cu at (247.4, 48.9)
- added D37: 1N4148W, Diode_SMD:D_SOD-123, F.Cu at (106.7, 170.1)
- added D38: 1N4148W, Diode_SMD:D_SOD-123, F.Cu at (221.5, 89.3)
- added D39: 1N4148W, Diode_SMD:D_SOD-123, F.Cu at (112.5, 170.1)
- added D4: 1N4148W, Diode_SMD:D_SOD-123, F.Cu at (247.4, 62.3)
- added D40: 1N4148W, Diode_SMD:D_SOD-123, F.Cu at (66.5, 170.1)
- added D41: 1N4148W, Diode_SMD:D_SOD-123, F.Cu at (55.0, 170.1)
- added D42: 1N4148W, Diode_SMD:D_SOD-123, F.Cu at (129.7, 170.1)
- added D43: 1N4148W, Diode_SMD:D_SOD-123, F.Cu at (118.2, 170.1)
- added D44: 1N4148W, Diode_SMD:D_SOD-123, F.Cu at (124.0, 170.1)
- added D45: 1N4148W, Diode_SMD:D_SOD-123, F.Cu at (227.2, 79.4)
- added D46: 1N4148W, Diode_SMD:D_SOD-123, F.Cu at (72.2, 173.4)
- added D47: 1N4148W, Diode_SMD:D_SOD-123, F.Cu at (83.7, 170.1)
- added D48: 1N4148W, Diode_SMD:D_SOD-123, F.Cu at (247.4, 58.9)
- added D49: 1N4148W, Diode_SMD:D_SOD-123, F.Cu at (253.2, 48.9)
- added D5: 1N4148W, Diode_SMD:D_SOD-123, F.Cu at (66.5, 173.4)
- added D6: 1N4148W, Diode_SMD:D_SOD-123, F.Cu at (78.0, 170.1)
- added D7: 1N4148W, Diode_SMD:D_SOD-123, F.Cu at (207.0, 103.7)
- added D8: 1N4148W, Diode_SMD:D_SOD-123, F.Cu at (106.7, 173.4)
- added D9: 1N4148W, Diode_SMD:D_SOD-123, F.Cu at (89.5, 173.4)
- added E1: MX-NoLED, MX_Alps_Hybrid:MX-1U-NoLED, F.Cu at (133.4, 77.5)
- added Enter1: MX-NoLED, MX_Alps_Hybrid:MX-1U-NoLED, F.Cu at (93.0, 97.7)
- added F1: 500mA, Fuse:Fuse_1206_3216Metric, F.Cu at (258.8, 52.2)
- added F2: MX-NoLED, MX_Alps_Hybrid:MX-1U-NoLED, F.Cu at (113.2, 158.3)
- added Fn1: MX-NoLED, MX_Alps_Hybrid:MX-1U-NoLED, F.Cu at (133.4, 138.1)
- added G1: MX-NoLED, MX_Alps_Hybrid:MX-1U-NoLED, F.Cu at (72.8, 97.7)
- added H1: MX-NoLED, MX_Alps_Hybrid:MX-1U-NoLED, F.Cu at (72.8, 57.3)
- added I1: MX-NoLED, MX_Alps_Hybrid:MX-1U-NoLED, F.Cu at (113.2, 117.9)
- added J1: MX-NoLED, MX_Alps_Hybrid:MX-1U-NoLED, F.Cu at (133.4, 117.9)
- added K1: MX-NoLED, MX_Alps_Hybrid:MX-1U-NoLED, F.Cu at (93.0, 77.5)
- added L1: MX-NoLED, MX_Alps_Hybrid:MX-1U-NoLED, F.Cu at (113.2, 77.5)
- added M1: MX-NoLED, MX_Alps_Hybrid:MX-1U-NoLED, F.Cu at (133.4, 57.3)
- added Mod-1: MX-NoLED, MX_Alps_Hybrid:MX-1U-NoLED, F.Cu at (93.0, 117.9)
- added Mod-2: MX-NoLED, MX_Alps_Hybrid:MX-1U-NoLED, F.Cu at (113.2, 97.7)
- added Mod-Long1: MX-NoLED, MX_Alps_Hybrid:MX-1U-NoLED, F.Cu at (52.6, 117.9)
- added N1: MX-NoLED, MX_Alps_Hybrid:MX-1U-NoLED, F.Cu at (153.6, 138.1)
- added O1: MX-NoLED, MX_Alps_Hybrid:MX-1U-NoLED, F.Cu at (52.6, 158.3)
- added P1: MX-NoLED, MX_Alps_Hybrid:MX-1U-NoLED, F.Cu at (133.4, 158.3)
- added Q1: MX-NoLED, MX_Alps_Hybrid:MX-1U-NoLED, F.Cu at (153.6, 117.9)
- added R1: 22, Resistor_SMD:R_0805_2012Metric, F.Cu at (232.3, 82.1)
- added R2: 22, Resistor_SMD:R_0805_2012Metric, F.Cu at (226.5, 85.9)
- added R3: 10k, Resistor_SMD:R_0805_2012Metric, F.Cu at (252.5, 61.7)
- added R4: 10k, Resistor_SMD:R_0805_2012Metric, F.Cu at (232.3, 79.2)
- added R5: MX-NoLED, MX_Alps_Hybrid:MX-1U-NoLED, F.Cu at (173.8, 97.7)
- added S1: MX-NoLED, MX_Alps_Hybrid:MX-1U-NoLED, F.Cu at (173.8, 77.5)
- added SW1: SW_PUSH, random-keyboard-parts:SKQG-1155865, F.Cu at (47.3, 171.6)
- added Shift_L1: MX-NoLED, MX_Alps_Hybrid:MX-1U-NoLED, F.Cu at (214.2, 57.3)
- added Shift_R1: MX-NoLED, MX_Alps_Hybrid:MX-1U-NoLED, F.Cu at (93.0, 57.3)
- added Space1: MX-NoLED, MX_Alps_Hybrid:MX-1U-NoLED, F.Cu at (72.8, 138.1)
- added T1: MX-NoLED, MX_Alps_Hybrid:MX-1U-NoLED, F.Cu at (194.0, 97.7)
- added Tab1: MX-NoLED, MX_Alps_Hybrid:MX-1U-NoLED, F.Cu at (194.0, 77.5)
- added U1: ATmega32U4-A, Package_QFP:TQFP-44_10x10mm_P0.8mm, F.Cu at (211.4, 94.8)
- added U2: MX-NoLED, MX_Alps_Hybrid:MX-1U-NoLED, F.Cu at (52.6, 77.5)
- added USB1: Molex-0548190589, random-keyboard-parts:Molex-0548190589, F.Cu at (228.7, 72.6)
- added V1: MX-NoLED, MX_Alps_Hybrid:MX-1U-NoLED, F.Cu at (153.6, 77.5)
- added W1: MX-NoLED, MX_Alps_Hybrid:MX-1U-NoLED, F.Cu at (72.8, 77.5)
- added Win1: MX-NoLED, MX_Alps_Hybrid:MX-1U-NoLED, F.Cu at (173.8, 57.3)
- added Win2: MX-NoLED, MX_Alps_Hybrid:MX-1U-NoLED, F.Cu at (234.4, 57.3)
- added X1: MX-NoLED, MX_Alps_Hybrid:MX-1U-NoLED, F.Cu at (72.8, 117.9)
- added Y1: 16MHz, Crystal:Crystal_SMD_3225-4Pin_3.2x2.5mm, F.Cu at (243.4, 69.6)
- added Y2: MX-NoLED, MX_Alps_Hybrid:MX-1U-NoLED, F.Cu at (52.6, 57.3)
- added Z1: MX-NoLED, MX_Alps_Hybrid:MX-1U-NoLED, F.Cu at (214.2, 77.5)
- added [1: MX-NoLED, MX_Alps_Hybrid:MX-1U-NoLED, F.Cu at (194.0, 57.3)
- added \1: MX-NoLED, MX_Alps_Hybrid:MX-1U-NoLED, F.Cu at (153.6, 97.7)
- added ]1: MX-NoLED, MX_Alps_Hybrid:MX-1U-NoLED, F.Cu at (113.2, 57.3)
