File: pcb/rabid40/rabid40.kicad_pcb (KiCad board)
At the start: 2 copper layers, 112 parts, among them J1 MX-NoLED, K1 MX-NoLED, M1 MX-NoLED, P1 MX-NoLED, Q1 MX-NoLED, SW1 SW_PUSH, T1 MX-NoLED, U1 ATmega32U4-A, U2 MX-NoLED, X1 MX-NoLED, Y1 16MHz, Y2 MX-NoLED

Commit message: added multilayout support to schematic
Parts:
- moved O1 197.3 mm to (199.2, 26.2)
- moved Caps1 181.4 mm to (27.8, 45.2)
- moved Tab1 174.0 mm to (27.8, 26.2)
- moved /1 172.0 mm to (277.0, 85.7)
- moved P1 157.0 mm to (218.3, 26.2)
- moved A1 155.5 mm to (46.8, 45.2)
- moved ]1 146.5 mm to (256.4, 26.2)
- moved Q1 140.8 mm to (46.8, 26.2)
- moved U2 120.0 mm to (161.1, 26.2)
- moved I1 113.6 mm to (180.2, 26.2)
- moved S1 112.7 mm to (65.9, 45.2)
- moved T1 100.8 mm to (123.0, 26.2)
- moved R5 100.0 mm to (104.0, 26.2)
- moved Y2 94.7 mm to (142.1, 26.2)
- moved D17 93.2 mm to (84.9, 45.2)
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Changed lines of the file:
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@@
   )
   (footprint "MX_Alps_Hybrid:MX-1U-NoLED" (layer "F.Cu")
-    (at 153.63125 117.9125)
+    (at 46.83125 26.19375)
     (property "Sheetfile" "rabid40.kicad_sch")
     (property "Sheetname" "")
@@
   )
   (footprint "MX_Alps_Hybrid:MX-1U-NoLED" (layer "F.Cu")
-    (at 52.63125 77.5125)
+    (at 161.13125 26.19375)
     (property "Sheetfile" "rabid40.kicad_sch")
     (property "Sheetname" "")
@@
   )
   (footprint "MX_Alps_Hybrid:MX-1U-NoLED" (layer "F.Cu")
-    (at 113.23125 57.3125)
+    (at 256.38125 26.19375)
     (property "Sheetfile" "rabid40.kicad_sch")
     (property "Sheetname" "")
@@
   )
   (footprint "MX_Alps_Hybrid:MX-1U-NoLED" (layer "F.Cu")
-    (at 194.03125 57.3125)
+    (at 237.33125 26.19375)
     (property "Sheetfile" "rabid40.kicad_sch")
     (property "Sheetname" "")
@@
   )
   (footprint "MX_Alps_Hybrid:MX-1U-NoLED" (layer "F.Cu")
-    (at 52.63125 57.3125)
+    (at 142.08125 26.19375)
     (property "Sheetfile" "rabid40.kicad_sch")
     (property "Sheetname" "")
@@
   )
   (footprint "MX_Alps_Hybrid:MX-1U-NoLED" (layer "F.Cu")
-    (at 194.03125 117.9125)
+    (at 27.78125 45.24375)
     (property "Sheetfile" "rabid40.kicad_sch")
     (property "Sheetname" "")
@@
   )
   (footprint "MX_Alps_Hybrid:MX-1U-NoLED" (layer "F.Cu")
-    (at 173.83125 77.5125)
+    (at 65.88125 45.24375)
     (property "Sheetfile" "rabid40.kicad_sch")
     (property "Sheetname" "")
@@
   )
   (footprint "MX_Alps_Hybrid:MX-1U-NoLED" (layer "F.Cu")
-    (at 113.23125 138.1125)
+    (at 277.01875 85.725)
     (property "Sheetfile" "rabid40.kicad_sch")
     (property "Sheetname" "")
@@
   )
   (footprint "MX_Alps_Hybrid:MX-1U-NoLED" (layer "F.Cu")
-    (at 113.23125 117.9125)
+    (at 180.18125 26.19375)
     (property "Sheetfile" "rabid40.kicad_sch")
     (property "Sheetname" "")
@@
   )
   (footprint "MX_Alps_Hybrid:MX-1U-NoLED" (layer "F.Cu")
-    (at 93.03125 57.3125)
+    (at 65.88125 73.81875)
     (property "Sheetfile" "rabid40.kicad_sch")
     (property "Sheetname" "")
@@
   )
   (footprint "MX_Alps_Hybrid:MX-1U-NoLED" (layer "F.Cu")
-    (at 173.83125 138.1125)
+    (at 189.70625 138.1125)
     (property "Sheetfile" "rabid40.kicad_sch")
     (property "Sheetname" "")
@@
   )
   (footprint "MX_Alps_Hybrid:MX-1U-NoLED" (layer "F.Cu")
-    (at 153.63125 158.3125)
+    (at 46.83125 45.24375)
     (property "Sheetfile" "rabid40.kicad_sch")
     (property "Sheetname" "")
@@
   )
   (footprint "MX_Alps_Hybrid:MX-1U-NoLED" (layer "F.Cu")
-    (at 194.03125 97.7125)
+    (at 123.03125 26.19375)
     (property "Sheetfile" "rabid40.kicad_sch")
     (property "Sheetname" "")
@@
   )
   (footprint "MX_Alps_Hybrid:MX-1U-NoLED" (layer "F.Cu")
-    (at 93.03125 138.1125)
+    (at 84.93125 45.24375)
     (property "Sheetfile" "rabid40.kicad_sch")
     (property "Sheetname" "")
@@
   )
   (footprint "MX_Alps_Hybrid:MX-1U-NoLED" (layer "F.Cu")
-    (at 72.83125 57.3125)
+    (at 42.06875 73.025)
     (property "Sheetfile" "rabid40.kicad_sch")
     (property "Sheetname" "")
@@
   )
   (footprint "MX_Alps_Hybrid:MX-1U-NoLED" (layer "F.Cu")
-    (at 173.83125 97.7125)
+    (at 103.98125 26.19375)
     (property "Sheetfile" "rabid40.kicad_sch")
     (property "Sheetname" "")
@@
   )
   (footprint "MX_Alps_Hybrid:MX-1U-NoLED" (layer "F.Cu")
-    (at 133.43125 77.5125)
+    (at 84.93125 26.19375)
     (property "Sheetfile" "rabid40.kicad_sch")
     (property "Sheetname" "")
@@
   )
   (footprint "MX_Alps_Hybrid:MX-1U-NoLED" (layer "F.Cu")
-    (at 133.43125 158.3125)
+    (at 218.28125 26.19375)
     (property "Sheetfile" "rabid40.kicad_sch")
     (property "Sheetname" "")
@@
   )
   (footprint "MX_Alps_Hybrid:MX-1U-NoLED" (layer "F.Cu")
-    (at 72.83125 77.5125)
+    (at 65.88125 26.19375)
     (property "Sheetfile" "rabid40.kicad_sch")
     (property "Sheetname" "")
@@
   )
   (footprint "MX_Alps_Hybrid:MX-1U-NoLED" (layer "F.Cu")
-    (at 194.03125 77.5125)
+    (at 27.78125 26.19375)
     (property "Sheetfile" "rabid40.kicad_sch")
     (property "Sheetname" "")
@@
   )
   (footprint "MX_Alps_Hybrid:MX-1U-NoLED" (layer "F.Cu")
-    (at 52.63125 158.3125)
+    (at 199.23125 26.19375)
     (property "Sheetfile" "rabid40.kicad_sch")
     (property "Sheetname" "")

Commit message: more switches aligned
Parts:
- removed Space1: MX-NoLED, MX_Alps_Hybrid:MX-1U-NoLED
- added Alt3: MX-NoLED, MX_Alps_Hybrid:MX-1.5U, F.Cu at (-268.5, 143.0)
- added Mod-3: MX-NoLED, MX_Alps_Hybrid:MX-1U, F.Cu at (-88.8, 60.2)
- added Shift_Long1: MX-NoLED, MX_Alps_Hybrid:MX-2.75U, F.Cu at (-122.1, 19.8)
- added Space2.25: MX-NoLED, MX_Alps_Hybrid:MX-2.25U, F.Cu at (-141.1, 40.7)
- added Space6.25: MX-NoLED, MX_Alps_Hybrid:MX-6.25U, F.Cu at (-223.2, 40.7)
- added Space7: MX-NoLED, MX_Alps_Hybrid:MX-7U, F.Cu at (-216.1, 19.8)
- added SteppedCaps1: MX-NoLED, MX_Alps_Hybrid:MX-1U, F.Cu at (-159.1, 101.9)
- added Win3: MX-NoLED, MX_Alps_Hybrid:MX-1.25U, F.Cu at (-270.9, 163.2)
- added Win4: MX-NoLED, MX_Alps_Hybrid:MX-1U, F.Cu at (-199.5, 102.6)
- '1, /1, ;1, <1, >1, A1, B1, C8, D17, E1, F2, Fn1, G1, H1, I1, J1, K1, L1, M1, Mod-1, Mod-2, N1, O1, P1, Q1, R5, S1, T1, U2, V1, W1, Win1, X1, Y2, Z1, [1, ]1: footprint MX_Alps_Hybrid:MX-1U-NoLED -> MX_Alps_Hybrid:MX-1U
- Alt1, Tab1, \1: footprint MX_Alps_Hybrid:MX-1U-NoLED -> MX_Alps_Hybrid:MX-1.5U
- Alt2, Win2: footprint MX_Alps_Hybrid:MX-1U-NoLED -> MX_Alps_Hybrid:MX-1.25U
- Caps1, Shift_R1: footprint MX_Alps_Hybrid:MX-1U-NoLED -> MX_Alps_Hybrid:MX-1.75U
- Enter1, Shift_L1: footprint MX_Alps_Hybrid:MX-1U-NoLED -> MX_Alps_Hybrid:MX-2.25U
- Mod-Long1: footprint MX_Alps_Hybrid:MX-1U-NoLED -> MX_Alps_Hybrid:MX-2.75U
- moved C3 500.3 mm to (-262.2, 104.9)
- moved USB1 493.9 mm to (-264.6, 98.3)
- moved D16 493.7 mm to (-254.5, 108.2)
- moved U1 487.5 mm to (-276.1, 100.3)
- moved Z1 470.4 mm to (-248.3, 163.2)
- moved C5 431.9 mm to (-165.8, 137.4)
- moved /1 431.8 mm to (-153.2, 122.1)
- moved C4 425.1 mm to (-165.8, 134.4)
- moved R3 413.9 mm to (-149.4, 160.6)
- moved D32 408.2 mm to (-143.0, 154.1)
- moved Win2 407.8 mm to (-173.3, 61.5)
- moved D4 406.7 mm to (-148.8, 154.1)
- moved R4 404.3 mm to (-165.9, 149.4)
- moved D18 401.5 mm to (-154.5, 154.1)
- moved D26 389.6 mm to (-154.5, 160.8)
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Connections:
- Alt1 pad 2: Net-(Alt1-Pad2) -> Net-(D8-Pad2)
- Alt2 pad 1: Col 6 -> Col 1
- Alt2 pad 2: Net-(Alt2-Pad2) -> Net-(D8-Pad2)
- D29 pad 2: Net-(Alt2-Pad2) -> Net-(Alt3-Pad2)
- D33 pad 2: Net-(Win2-Pad2) -> Net-(D33-Pad2)
- D5 pad 2: Net-(Win1-Pad2) -> Net-(Win2-Pad2)
- D8 pad 2: Net-(Alt1-Pad2) -> Net-(D8-Pad2)
- Mod-2 pad 1: Col 5 -> Col 6
- Mod-Long1 pad 1: Col 4 -> Col 5
- Win1 pad 2: Net-(Win1-Pad2) -> Net-(Win2-Pad2)
- Win2 pad 1: Col 7 -> Col 0

Commit message: switches in order, mcu components near their place
Parts:
- removed Alt2, Win2, Win3: MX-NoLED, MX_Alps_Hybrid:MX-1.25U
- removed Mod-3: MX-NoLED, MX_Alps_Hybrid:MX-1U
- removed Space6.25: MX-NoLED, MX_Alps_Hybrid:MX-6.25U
- Mod-Long1: footprint MX_Alps_Hybrid:MX-2.75U -> MX_Alps_Hybrid:MX-2.75U-ReversedStabilizers
- Space2.25: footprint MX_Alps_Hybrid:MX-2.25U -> MX_Alps_Hybrid:MX-2.25U-ReversedStabilizers
- Space7: footprint MX_Alps_Hybrid:MX-7U -> MX_Alps_Hybrid:MX-7U-ReversedStabilizers
- USB1: value Molex-0548190589 -> JST_SH_SM04B-SRSS-TB_1x04-1MP_P1.00mm_Horizontal; footprint random-keyboard-parts:Molex-0548190589 -> Connector_JST:JST_SH_SM04B-SRSS-TB_1x04-1MP_P1.00mm_Horizontal
- moved D47 622.1 mm to (355.6, 133.3), turned to 90 degrees
- moved Enter1 598.5 mm to (335.0, 133.3)
- moved D46 588.1 mm to (327.8, 114.3), turned to 90 degrees
- moved Alt3 563.7 mm to (294.5, 171.4)
- moved D43 563.4 mm to (308.0, 114.3), turned to 90 degrees
- moved D29 555.6 mm to (303.2, 171.4), turned to 90 degrees
- moved D41 540.9 mm to (293.7, 133.3), turned to 90 degrees
- moved D40 532.9 mm to (288.9, 114.3), turned to 90 degrees
- moved Win4 522.4 mm to (318.3, 171.4)
- moved Shift_R1 513.1 mm to (320.7, 152.4)
- moved Mod-Long1 503.7 mm to (234.9, 171.4)
- moved D30 477.8 mm to (231.8, 114.3), turned to 90 degrees
- moved <1 475.0 mm to (256.4, 152.4)
- moved Shift_Long1 471.3 mm to (330.2, 152.4)
- moved D20 465.6 mm to (188.9, 152.4), turned to 90 degrees
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
Commit message: repositioned capacitors
Parts:
- C7: value 0.1uF -> 10uF
- Mod-Long1: footprint MX_Alps_Hybrid:MX-2.75U-ReversedStabilizers -> MX_Alps_Hybrid:MX-2.75U
- Space2.25: footprint MX_Alps_Hybrid:MX-2.25U-ReversedStabilizers -> MX_Alps_Hybrid:MX-2.25U
- Space7: footprint MX_Alps_Hybrid:MX-7U-ReversedStabilizers -> MX_Alps_Hybrid:MX-7U
- moved C5 25.2 mm to (65.9, 154.9)
- moved R4 24.8 mm to (66.7, 171.6), turned to -90 degrees
- moved C1 22.5 mm to (43.5, 157.2)
- moved C2 19.6 mm to (58.6, 140.5), turned to 0 degrees
- moved C7 17.2 mm to (51.0, 140.5), turned to 180 degrees
- moved R3 12.0 mm to (43.5, 161.1)
- moved C6 10.9 mm to (43.7, 149.9)
- moved SteppedCaps1 3.17 mm to (84.1, 152.4)
- moved Y1 0.31 mm to (54.5, 161.9), turned to 180 degrees
Connections:
- U1 pad 10: unconnected-(U1-Pad10) -> Col2
- U1 pad 11: unconnected-(U1-Pad11) -> Col3
- U1 pad 12: unconnected-(U1-Pad12) -> Col7
- U1 pad 18: unconnected-(U1-Pad18) -> Col10
- U1 pad 19: unconnected-(U1-Pad19) -> Col11
- U1 pad 20: unconnected-(U1-Pad20) -> Col12
- U1 pad 21: unconnected-(U1-Pad21) -> Col13
- U1 pad 22: unconnected-(U1-Pad22) -> Row2
- U1 pad 25: unconnected-(U1-Pad25) -> Row3
- U1 pad 26: unconnected-(U1-Pad26) -> Row1
- U1 pad 27: unconnected-(U1-Pad27) -> Row0
- U1 pad 28: unconnected-(U1-Pad28) -> Col4
- U1 pad 29: unconnected-(U1-Pad29) -> Col5
- U1 pad 30: unconnected-(U1-Pad30) -> Col6
- U1 pad 31: unconnected-(U1-Pad31) -> Col8
- U1 pad 32: unconnected-(U1-Pad32) -> Col9
- U1 pad 8: unconnected-(U1-Pad8) -> Col0
- U1 pad 9: unconnected-(U1-Pad9) -> Col1
