File: pcb/rabid40/rabid40.kicad_pcb (KiCad board)
At the start: 2 copper layers, 136 parts, among them J1 SWD, J2 Conn_01x04, J3 MX_SW_solder, K1 MX_SW_solder, M1 MX_SW_solder, P1 MX_SW_solder, Q1 MX_SW_solder, SW7 SW_Push, T1 MX_SW_solder, U1 RP2040, U2 W25Q128JVS, U3 XC6206PxxxMR-Regulator_Linear, U4 MX_SW_solder, X1 MX_SW_solder, Y1 12MHz, Y2 MX_SW_solder

Commit message: moved some mcu components into place
Parts:
- C1, C10, C11, C12, C13, C14, C15, C16, C17, C2, C3, C4, C5, C6, C7, C8, C9, D1, D10, D11, D12, D13, D14, D15, D16, D17, D18, D19, D2, D20, D21, D22, D23, D24, D25, D26, D27, D28, D29, D3, D30, D31, D32, D33, D34, D35, D36, D37, D38, D39, D4, D40, D41, D42, D43, D44, D47, D48, D49, D5, D50, D52, D6, D7, D8, D9, F1, R1, R2, R3, R4, R5, U1, U2, U3, Y1: moved to B.Cu
- J2: footprint Connector_JST:JST_EH_S4B-EH_1x04_P2.50mm_Horizontal -> Connector_JST:JST_SH_SM04B-SRSS-TB_1x04-1MP_P1.00mm_Horizontal; moved to B.Cu
- SW7: footprint Connector_PinSocket_2.54mm:PinSocket_1x02_P2.54mm_Vertical -> Button_Switch_SMD:SW_SPST_TL3342; moved to B.Cu
- moved C7 307.7 mm to (-36.3, 19.4), turned to 180 degrees
- moved U3 292.0 mm to (-27.8, 36.5), turned to 180 degrees
- moved C6 289.7 mm to (-44.5, 51.6), turned to 180 degrees
- moved C8 286.9 mm to (-25.3, 18.9), turned to 180 degrees
- moved Y1 281.1 mm to (-30.2, 46.8), turned to 180 degrees
- moved C4 277.3 mm to (-11.0, 15.4), turned to 180 degrees
- moved C9 272.2 mm to (-8.16, 15.4), turned to 180 degrees
- moved C10 256.7 mm to (-16.7, 52.5), turned to -90 degrees
- moved C2 255.1 mm to (-16.7, 49.6), turned to -90 degrees
- moved C17 253.5 mm to (-16.7, 46.7), turned to -90 degrees
- moved C3 252.0 mm to (-16.7, 43.8), turned to -90 degrees
- moved C14 249.2 mm to (-16.7, 38.1), turned to -90 degrees
- moved C15 245.4 mm to (-16.7, 29.5), turned to -90 degrees
- moved C12 244.3 mm to (-16.7, 26.6), turned to -90 degrees
- moved C13 243.2 mm to (-16.7, 23.8), turned to -90 degrees
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
Commit message: started placing traces, its very scuff
Parts:
- moved C8 154.4 mm to (111.7, 89.9), turned to 90 degrees
- moved U2 153.5 mm to (117.3, 92.3)
- moved C7 153.2 mm to (93.9, 100.1)
- moved C16 152.8 mm to (105.5, 112.6)
- moved C6 148.1 mm to (96.5, 96.9), turned to 90 degrees
- moved Y1 147.8 mm to (102.3, 112.2), turned to 0 degrees
- moved C12 145.5 mm to (106.3, 104.4), turned to -45 degrees
- moved R5 143.3 mm to (100.6, 109.2), turned to 90 degrees
- moved C13 142.9 mm to (105.2, 98.4), turned to 90 degrees
- moved C14 136.1 mm to (99.4, 109.2)
- moved C9 134.5 mm to (99.3, 96.4), turned to 90 degrees
- moved C17 133.5 mm to (99.7, 112.1), turned to 90 degrees
- moved C2 129.6 mm to (98.4, 109.2)
- moved R2 129.5 mm to (95.8, 74.0)
- moved R1 129.3 mm to (97.6, 74.1)
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Routing:
- net +3V3: track 0.00 -> 166.8 mm, vias 0 -> 1
- net Row3: track 0.00 -> 53.4 mm
- net CS: track 0.00 -> 35.1 mm
- net SD1: track 0.00 -> 33.2 mm
- net SD2: track 0.00 -> 31.8 mm
- net GND: track 0.00 -> 23.0 mm, vias 0 -> 8
- net SD3: track 0.00 -> 18.6 mm
- net QSPI_CLK: track 0.00 -> 17.6 mm
- net SD0: track 0.00 -> 17.3 mm
- net XTAL_IN: track 0.00 -> 11.5 mm
- net Net-(D10-Pad2): track 0.00 -> 7.94 mm
- net Net-(Alt1-Pad2): track 0.00 -> 7.94 mm
- net +1V1: track 0.00 -> 6.86 mm, vias 0 -> 1
- net Net-(D18-Pad2): track 0.00 -> 5.79 mm
- net /D_-: track 0.00 -> 3.57 mm
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- added copper zone on B.Cu, net +1V1
- added copper zone on B.Cu, net +3V3

Commit message: completed routing
Parts:
- Alt1, Alt2: footprint marbastlib-mx:SW_MX_1.5u -> marbastlib-mx:SW_MX_1u
- J2: footprint Connector_JST:JST_SH_SM04B-SRSS-TB_1x04-1MP_P1.00mm_Horizontal -> Connector_JST:JST_EH_S4B-EH_1x04_P2.50mm_Horizontal
- SW7: footprint Button_Switch_SMD:SW_SPST_TL3342 -> Connector_PinSocket_2.54mm:PinSocket_1x02_P2.54mm_Vertical
- Shift2: footprint marbastlib-mx:SW_MX_1.75u -> marbastlib-mx:SW_MX_1u
- moved J1 84.3 mm to (75.3, 94.5), turned to -90 degrees
- moved R3 83.5 mm to (74.8, 99.0), turned to 0 degrees
- moved R4 72.4 mm to (123.1, 89.6)
- moved SW7 70.7 mm to (123.6, 84.8), turned to 180 degrees
- moved D2 24.7 mm to (31.1, 66.7)
- moved R1 15.5 mm to (100.5, 58.9), turned to 180 degrees
- moved R2 14.4 mm to (100.5, 60.3), turned to 180 degrees
- moved J2 3.83 mm to (112.7, 61.4), turned to 90 degrees
- moved C9 1.32 mm to (99.2, 95.1)
- moved C1 1.31 mm to (100.2, 95.1)
- moved C10 1.24 mm to (95.1, 103.8)
- moved C12 0.61 mm to (106.9, 104.4), turned to 0 degrees
- moved C14 0.26 mm to (99.4, 109.5)
- moved C2 0.18 mm to (98.4, 109.4)
Connections:
- J2 pad 2: D_USB_N -> D_N
- J2 pad 3: D_USB_P -> D_P
- U1 pad 11: unconnected-(U1-Pad11) -> Col13
- U1 pad 2: Col0 -> Col5
- U1 pad 27: unconnected-(U1-Pad27) -> Col0
- U1 pad 28: unconnected-(U1-Pad28) -> Col1
- U1 pad 29: unconnected-(U1-Pad29) -> Col2
- U1 pad 3: Col1 -> Col6
- U1 pad 30: unconnected-(U1-Pad30) -> Row1
- U1 pad 35: unconnected-(U1-Pad35) -> Col4
- U1 pad 36: unconnected-(U1-Pad36) -> Col3
- U1 pad 38: unconnected-(U1-Pad38) -> Row3
- U1 pad 39: unconnected-(U1-Pad39) -> Row2
- U1 pad 4: Col3 -> Col7
- U1 pad 41: unconnected-(U1-Pad41) -> Row0
- U1 pad 5: Col4 -> Col8
- U1 pad 6: unconnected-(U1-Pad6) -> Col9
- U1 pad 7: unconnected-(U1-Pad7) -> Col10
- U1 pad 8: unconnected-(U1-Pad8) -> Col11
- U1 pad 9: unconnected-(U1-Pad9) -> Col12
Routing:
- net Row2: track 0.00 -> 324.6 mm, vias 0 -> 2
- net Row0: track 0.00 -> 321.4 mm, vias 0 -> 2
- net Row1: track 0.00 -> 303.7 mm, vias 0 -> 4
- net Col12: track 0.00 -> 267.4 mm, vias 0 -> 1
- net Col13: track 0.00 -> 256.0 mm, vias 0 -> 1
- net Col10: track 0.00 -> 252.4 mm, vias 0 -> 1
- net Col11: track 0.00 -> 222.9 mm, vias 0 -> 3
- net Col9: track 0.00 -> 213.8 mm, vias 0 -> 1
- net Row3: track 53.4 -> 247.2 mm, vias 0 -> 2
- net Col8: track 0.00 -> 184.1 mm, vias 0 -> 1
- net Col2: track 0.00 -> 183.9 mm, vias 0 -> 1
- net Col1: track 0.00 -> 173.7 mm, vias 0 -> 1
- net Col0: track 0.00 -> 162.6 mm, vias 0 -> 2
- net Col3: track 0.00 -> 151.4 mm, vias 0 -> 3
- net Col7: track 0.00 -> 147.2 mm
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
Commit message: finished routing
Parts:
- Alt1, Alt2: footprint marbastlib-mx:SW_MX_1u -> marbastlib-mx:SW_MX_1.5u
- J2: moved to F.Cu
- moved R1 21.3 mm to (116.4, 72.9), turned to -90 degrees
- moved R2 19.1 mm to (114.9, 72.9), turned to -90 degrees
- moved C10 2.44 mm to (92.7, 103.8)
- moved J2 2.38 mm to (113.6, 59.2), turned to 0 degrees
- moved D16 1.03 mm to (111.7, 68.6)
- moved D42 0.58 mm to (259.0, 105.8)
- moved C16 0.16 mm to (105.3, 112.6)
Routing:
- net /D_+: track 47.7 -> 33.9 mm, vias 2 -> 0
- net /D_-: track 47.1 -> 33.5 mm, vias 2 -> 0
- net +3V3: track 133.0 -> 135.4 mm
- net VBUS: track 11.9 -> 10.3 mm, vias 2 -> 0
- net D_N: track 12.1 -> 13.5 mm
- net D_P: track 12.5 -> 13.9 mm
- net Row1: track 303.7 -> 305.0 mm, vias 4 -> 6
- net Net-(D16-Pad2): track 8.27 -> 7.10 mm
- net GND: track 25.4 -> 24.3 mm, vias 9 -> 8
- net Row3: track 247.2 -> 246.6 mm
- net Row2: vias 2 -> 4
- added copper zone on B.Cu, net GND
Other:
- board outline added: 285.8 x 76.2 mm

Commit message: added annotationos
Other:
- board text added: "1"
- board text added: "2022/08/10"
- board text added: "Rabid40"
Changed lines of the file:
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@@
   (gr_arc (start 289.475 38.4) (mid 289.669454 38.480546) (end 289.75 38.675) (layer "Edge.Cuts") (width 0.1))
   (gr_line (start 31.505546 96.499454) (end 4.3 96.51) (layer "Edge.Cuts") (width 0.1))
+  (gr_text "1" (at 270 193.12) (layer "Margin")
+    (effects (font (size 1 1) (thickness 0.15)))
+  )
+  (gr_text "Rabid40" (at 195.62 189.63) (layer "Margin")
+    (effects (font (size 3 3) (thickness 0.15)))
+  )
+  (gr_text "2022/08/10" (at 211.95 193.01) (layer "Margin")
+    (effects (font (size 1 1) (thickness 0.15)))
+  )
   (via (at 117.28 92.3) (size 0.8) (drill 0.4) (layers "F.Cu" "B.Cu") (net 0))
   (segment (start 117.28 92.29) (end 117.28 92.3) (width 0.2) (layer "B.Cu") (net 0))

Commit message: pcb updated with feedback from tradesplatter. Gerbers regenerated
Routing:
- net GND: track 24.3 -> 38.0 mm, vias 8 -> 15
- net +1V1: track 19.5 -> 21.0 mm, vias 6 -> 4
- net CS: track 36.0 -> 34.9 mm
- net SD1: track 33.2 -> 32.2 mm
- net SD0: track 17.3 -> 16.2 mm
- net QSPI_CLK: track 17.6 -> 16.5 mm
- net SD2: track 31.8 -> 30.7 mm
- net SD3: track 18.6 -> 17.5 mm
- net (no net): track 0.01 -> 0.00 mm, vias 1 -> 0
- added copper zone on F.Cu, net GND
Other:
- outline, holes or cut-outs redrawn
- board text added: "Rabid40 v1 by Cujo26"
- board text added: "_ ,:'/ _..._ // ( `{dblquote}{dblquote}-.._.' \| / 6\___ | 6 4 | / \_ .--' (_'---'`) / `'---`() ,' | , .'` | )\ _.-' ; / | .'` _ / /` / .' '. , | / / / \ ; | | | \ | | .| | | \ `{dblquote}| /.-' | | | '-..-\ _.;.._ | |.;-. \ <`.._ )) | .;-. )) (__. ` ))-' \_ ))' `'--{dblquote}` `{dblquote}{dblquote}{dblquote}`"
