File: pcb/rabid40/_autosave-rabid40.kicad_pcb (KiCad board)
At the start: 2 copper layers, 112 parts, among them J1 MX-NoLED, K1 MX-NoLED, M1 MX-NoLED, P1 MX-NoLED, Q1 MX-NoLED, SW1 SW_PUSH, T1 MX-NoLED, U1 ATmega32U4-A, U2 MX-NoLED, X1 MX-NoLED, Y1 16MHz, Y2 MX-NoLED

Commit message: added multilayout support to schematic
Parts:
- removed '1, /1, ;1, <1, >1, A1, Alt1, Alt2, B1, C8, Caps1, D17, E1, Enter1, F2, Fn1, G1, H1, I1, J1, K1, L1, M1, Mod-1, Mod-2, Mod-Long1, N1, O1, P1, Q1, R5, S1, Shift_L1, Shift_R1, Space1, T1, Tab1, U2, V1, W1, Win1, Win2, X1, Y2, Z1, [1, \1, ]1: MX-NoLED, MX_Alps_Hybrid:MX-1U-NoLED
- removed C1, C2, C5, C7: 0.1uF, Capacitor_SMD:C_0805_2012Metric
- removed C3, C4: 22pF, Capacitor_SMD:C_0805_2012Metric
- removed C6: 1uF, Capacitor_SMD:C_0805_2012Metric
- removed D1, D10, D11, D12, D13, D14, D15, D16, D18, D19, D2, D20, D21, D22, D23, D24, D25, D26, D27, D28, D29, D3, D30, D31, D32, D33, D34, D35, D36, D37, D38, D39, D4, D40, D41, D42, D43, D44, D45, D46, D47, D48, D49, D5, D6, D7, D8, D9: 1N4148W, Diode_SMD:D_SOD-123
- removed F1: 500mA, Fuse:Fuse_1206_3216Metric
- removed R1, R2: 22, Resistor_SMD:R_0805_2012Metric
- removed R3, R4: 10k, Resistor_SMD:R_0805_2012Metric
- removed SW1: SW_PUSH, random-keyboard-parts:SKQG-1155865
- removed U1: ATmega32U4-A, Package_QFP:TQFP-44_10x10mm_P0.8mm
- removed USB1: Molex-0548190589, random-keyboard-parts:Molex-0548190589
- removed Y1: 16MHz, Crystal:Crystal_SMD_3225-4Pin_3.2x2.5mm
