File: pcb/rabid40/_autosave-rabid40.kicad_sch (KiCad schematic)
At the start: 115 parts, among them J1 MX-NoLED, K1 MX-NoLED, M1 MX-NoLED, P1 MX-NoLED, Q1 MX-NoLED, SW1 SW_PUSH, T1 MX-NoLED, U1 ATmega32U4-A, U2 MX-NoLED, X1 MX-NoLED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

Commit message: repositioned capacitors
Parts:
- C7: value 0.1uF -> 10uF
- USB1: footprint random-keyboard-parts:Molex-0548190589 -> Connector_JST:JST_SH_SM04B-SRSS-TB_1x04-1MP_P1.00mm_Horizontal
Changed lines of the file:
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@@
       (effects (font (size 1.27 1.27)) (justify right))
     )
-    (property "Value" "0.1uF" (id 1) (at 53.34 160.0135 0)
+    (property "Value" "10uF" (id 1) (at 53.34 160.0135 0)
       (effects (font (size 1.27 1.27)) (justify right))
     )
@@
       (effects (font (size 1.524 1.524)))
     )
-    (property "Footprint" "random-keyboard-parts:Molex-0548190589" (id 2) (at 22.86 27.94 0)
+    (property "Footprint" "Connector_JST:JST_SH_SM04B-SRSS-TB_1x04-1MP_P1.00mm_Horizontal" (id 2) (at 22.86 27.94 0)
       (effects (font (size 1.524 1.524)) hide)
     )
@@
     )
     (path "/210e289f-96fc-4fc6-b33a-b43e11937399"
-      (reference "C7") (unit 1) (value "0.1uF") (footprint "Capacitor_SMD:C_0805_2012Metric")
+      (reference "C7") (unit 1) (value "10uF") (footprint "Capacitor_SMD:C_0805_2012Metric")
     )
     (path "/99f1158c-a186-44bb-8404-6b7c95d451ec"
@@
     )
     (path "/6c8a0b0a-b301-4f30-9f42-89b6fb1987cd"
-      (reference "USB1") (unit 1) (value "Molex-0548190589") (footprint "random-keyboard-parts:Molex-0548190589")
+      (reference "USB1") (unit 1) (value "Molex-0548190589") (footprint "Connector_JST:JST_SH_SM04B-SRSS-TB_1x04-1MP_P1.00mm_Horizontal")
     )
     (path "/3a759d0f-a5c6-44f3-9a5c-7b0e3a8bcb7b"
